File: hw/sch_pcb/USBMOUNT01A.kicad_pcb (KiCad board)
At the start: 2 copper layers, 50 x 20 mm, 18 parts, among them J1 RJ45, P1 USB_C_Plug_USB2.0, U1 FT232RL, U2 USBLC6-2SC6

Commit message: minor changes
Parts:
- P1: value USB_C_Plug_USB2.0 -> USB_C
- moved C1 1.90 mm to (134.8, 82.4)
- moved C2 1.89 mm to (137.4, 82.4)
- moved R1 1.20 mm to (132.2, 82.4), turned to 90 degrees
- moved C3 0.26 mm to (135.9, 92.5)
Connections:
- JP1 pad 2: Net-(U1-Pad4) -> (no net)
- U1 pad 26: unconnected-(U1-Pad26) -> GND
- U1 pad 4: Net-(U1-Pad4) -> (no net)
Routing:
- net Net-(U1-Pad4): track 12.0 -> 0.00 mm
- net (no net): track 0.00 -> 12.0 mm
- net GND: track 0.00 -> 2.60 mm, vias 4 -> 5
- net +3V3: track 41.0 -> 39.1 mm
- net +5V: track 62.9 -> 61.7 mm

Commit message: update kicad version
Parts:
- P1: value USB_C -> USB4105-GF-A
Connections:
- JP1 pad 2: (no net) -> Net-(JP1-Pad2)
- U1 pad 4: (no net) -> Net-(JP1-Pad2)
Routing:
- net Net-(JP1-Pad2): track 0.00 -> 12.0 mm
- net (no net): track 12.0 -> 0.00 mm
- net /D+i: track 14.6 -> 11.7 mm
- net +5V: track 61.7 -> 60.4 mm
- net GND: track 2.60 -> 1.40 mm
- net +3V3: track 39.1 -> 38.0 mm

Commit message: resave to kicad7
Connections:
- net /D+i renamed /Di+
- net /D-i renamed /Di-
Routing:
- net Net-(JP1-C): track 12.0 -> 11.1 mm
- net /Di+: track 11.7 -> 12.3 mm
