File: hw/sch_pcb/USBMOUNT01A.kicad_sch (KiCad schematic)
At the start: 18 parts, among them J1 RJ45, P1 USB_C_Plug_USB2.0, U1 FT232RL, U2 USBLC6-2SC6

Commit message: minor changes
Connections:
- net GND: now also U1.26 (TEST)
Other:
- company: (none) -> AstroMeters
- title: (none) -> USBMOUNT01
- moved on the sheet: C1, C2, C3, D1, D2, D3, D4, J1, JP1, P1, R1, R3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

Commit message: update kicad version
Parts:
- P1: value USB_C_Plug_USB2.0 -> USB4105-GF-A; digikey (none) -> 2073-USB4105-GF-ACT-ND

Commit message: resave to kicad7
Connections:
- net D+i renamed Di+
- net D-i renamed Di-
- no-connect marks 0 -> 15
